Commit message: Add camera link.

File: bbot_description/urdf/bbot.xacro (robot description, xacro)
@@ -6,4 +6,6 @@
   <xacro:property name="woa" value="4" />
   <xacro:property name="doa" value="2" />
+  <xacro:property name="camera_mass" value="0.1" />
+  <xacro:property name="camera_size" value="0.1" />
   <!-- Import Gazebo elements -->
   <xacro:include filename="$(find bbot_description)/urdf/bbot.gazebo" />
@@ -32,3 +34,45 @@
     </inertial>
   </link>
+  <!-- Camera -->
+  <link name="camera_link">
+    <visual>
+      <geometry>
+        <box size="${camera_size} ${camera_size} ${camera_size}"/>
+      </geometry>
+      <material name="black" />
+    </visual>
+    <collision>
+      <geometry>
+        <box size="${camera_size} ${camera_size} ${camera_size}"/>
+      </geometry>
+    </collision>
+    <inertial>
+      <mass value="${camera_mass}" />
+      <inertia
+        ixx="${camera_mass * (camera_size * camera_size) / 6.0}" ixy="0.0" ixz="0.0"
+        iyy="${camera_mass * (camera_size * camera_size) / 6.0}" iyz="0.0"
+        izz="${camera_mass * (camera_size * camera_size) / 6.0}" />
+    </inertial>
+  </link>
+  <joint name="camera_joint" type="fixed">
+    <axis xyz="0 1 0" />
+    <origin xyz="0 0 ${doa}/2" rpy="0 0 0"/>
+    <parent link="base_link"/>
+    <child link="camera_link"/>
+  </joint>
+  <!--
+    generate an optical frame http://www.ros.org/reps/rep-0103.html#suffix-frames
+    so that ros and opencv can operate on the camera frame correctly
+  -->
+  <link name="camera_link_optical">
+  </link>
+  <joint name="camera_optical_joint" type="fixed">
+    <!--
+      these values have to be these values otherwise the gazebo camera image
+      won't be aligned properly with the frame it is supposedly originating from
+    -->
+    <origin xyz="0 0 0" rpy="${-pi/2} 0 ${-pi/2}"/>
+    <parent link="camera_link"/>
+    <child link="camera_link_optical"/>
+  </joint>
 </robot>

Commit message: Add various sensors to bbot: laser scan, gps, imu, magnetometer.

File: bbot_description/urdf/bbot.xacro (robot description, xacro)
@@ -18,6 +18,14 @@
   <xacro:property name="hull_woa" value="4.0" />
   <xacro:property name="hull_doa" value="2.0" />
-  <xacro:property name="camera_mass" value="0.1" />
-  <xacro:property name="camera_size" value="0.1" />
+  <xacro:property name="cam_mass" value="0.1" />
+  <xacro:property name="cam_size" value="0.1" />
+  <xacro:property name="ray_mass" value="0.1" />
+  <xacro:property name="ray_size" value="0.1" />
+  <xacro:property name="imu_mass" value="0.1" />
+  <xacro:property name="imu_size" value="0.1" />
+  <xacro:property name="gps_mass" value="0.1" />
+  <xacro:property name="gps_size" value="0.1" />
+  <xacro:property name="mag_mass" value="0.1" />
+  <xacro:property name="mag_size" value="0.1" />
   <!-- Import Gazebo elements -->
   <xacro:include filename="$(find bbot_description)/urdf/bbot.gazebo" />
@@ -40,23 +48,107 @@
   </link>
   <!-- Camera -->
-  <link name="camera_link">
+  <link name="cam_link">
     <visual>
       <geometry>
-        <box size="${camera_size} ${camera_size} ${camera_size}"/>
+        <box size="${cam_size} ${cam_size} ${cam_size}"/>
       </geometry>
-      <material name="black" />
+      <material name="red" />
     </visual>
     <collision>
       <geometry>
-        <box size="${camera_size} ${camera_size} ${camera_size}"/>
+        <box size="${cam_size} ${cam_size} ${cam_size}"/>
       </geometry>
     </collision>
-    <xacro:box_inertial mass="${camera_mass}" x="${camera_size}" y="${camera_size}" z="${camera_size}" />
+    <xacro:box_inertial mass="${cam_mass}" x="${cam_size}" y="${cam_size}" z="${cam_size}" />
   </link>
-  <joint name="camera_joint" type="fixed">
+  <joint name="cam_joint" type="fixed">
     <axis xyz="0 1 0" />
-    <origin xyz="${hull_loa/2 - 0.25} 0 ${hull_doa/2 + camera_size/2}" rpy="0 0 0"/>
+    <origin xyz="${hull_loa/2 - 0.25} 0 ${hull_doa/2 + cam_size/2}" rpy="0 0 0"/>
     <parent link="base_link"/>
-    <child link="camera_link"/>
+    <child link="cam_link"/>
+  </joint>
+  <!-- Ray -->
+  <link name="ray_link">
+    <visual>
+      <geometry>
+        <box size="${ray_size} ${ray_size} ${ray_size}"/>
+      </geometry>
+      <material name="red" />
+    </visual>
+    <collision>
+      <geometry>
+        <box size="${ray_size} ${ray_size} ${ray_size}"/>
+      </geometry>
+    </collision>
+    <xacro:box_inertial mass="${ray_mass}" x="${ray_size}" y="${ray_size}" z="${ray_size}" />
+  </link>
+  <joint name="ray_joint" type="fixed">
+    <axis xyz="0 1 0" />
+    <origin xyz="${hull_loa/2 - 0.25} 0.4 ${hull_doa/2 + ray_size/2}" rpy="0 0 0"/>
+    <parent link="base_link"/>
+    <child link="ray_link"/>
+  </joint>
+ <!-- GPS -->
+  <link name="gps_link">
+    <visual>
+      <geometry>
+        <box size="${gps_size} ${gps_size} ${gps_size}"/>
+      </geometry>
+      <material name="red" />
+    </visual>
+    <collision>
+      <geometry>
+        <box size="${gps_size} ${gps_size} ${gps_size}"/>
+      </geometry>
+    </collision>
+    <xacro:box_inertial mass="${gps_mass}" x="${gps_size}" y="${gps_size}" z="${gps_size}" />
+  </link>
+  <joint name="gps_joint" type="fixed">
+    <axis xyz="0 1 0" />
+    <origin xyz="0 0.4 ${hull_doa/2 + gps_size/2}" rpy="0 0 0"/>
+    <parent link="base_link"/>
+    <child link="gps_link"/>
+  </joint>
+ <!-- IMU -->
+  <link name="imu_link">
+    <visual>
+      <geometry>
+        <box size="${imu_size} ${imu_size} ${imu_size}"/>
+      </geometry>
+      <material name="red" />
+    </visual>
+    <collision>
+      <geometry>
+        <box size="${imu_size} ${imu_size} ${imu_size}"/>
+      </geometry>
+    </collision>
+    <xacro:box_inertial mass="${imu_mass}" x="${imu_size}" y="${imu_size}" z="${imu_size}" />
+  </link>
+  <joint name="imu_joint" type="fixed">
+    <axis xyz="0 1 0" />
+    <origin xyz="0 0 ${hull_doa/2 + imu_size/2}" rpy="0 0 0"/>
+    <parent link="base_link"/>
+    <child link="imu_link"/>
+  </joint>
+   <!-- Magnetometer -->
+  <link name="mag_link">
+    <visual>
+      <geometry>
+        <box size="${mag_size} ${mag_size} ${mag_size}"/>
+      </geometry>
+      <material name="red" />
+    </visual>
+    <collision>
+      <geometry>
+        <box size="${mag_size} ${mag_size} ${mag_size}"/>
+      </geometry>
+    </collision>
+    <xacro:box_inertial mass="${gps_mass}" x="${mag_size}" y="${mag_size}" z="${mag_size}" />
+  </link>
+  <joint name="mag_joint" type="fixed">
+    <axis xyz="0 1 0" />
+    <origin xyz="0 -0.4 ${hull_doa/2 + mag_size/2}" rpy="0 0 0"/>
+    <parent link="base_link"/>
+    <child link="mag_link"/>
   </joint>
 </robot>

File: bbot_description/urdf/materials.xacro (robot description, xacro)
@@ -3,4 +3,10 @@
   <material name="black">
     <color rgba="0.0 0.0 0.0 1.0"/>
+  </material>
+  <material name="red">
+    <color rgba="0.8 0.0 0.0 1.0"/>
+  </material>
+  <material name="green">
+    <color rgba="0.0 0.8 0.0 1.0"/>
   </material>
   <material name="blue">
